Commit message: added robot's second wheel

File: urdf/udacity_bot.xacro (robot description, xacro)
@@ -86,3 +86,34 @@
     </inertial>
 </link>
+<joint type="continuous" name="right_heel_hinge">
+    <origin xyz="0 -0.15 0" rpy="0 0 0"/>
+    <child link="right_wheel"/>
+    <parent link="chassis"/>
+    <axis xyz="0 1 0" rpy="0 0 0"/>
+    <limit effort="10000" velocity="1000"/>
+    <dynamics damping="1.0" friction="1.0"/>
+</joint>
+<link name="right_wheel">
+    <collision name="collision_right">
+        <origin xyz="0 0 0" rpy="0 -1.5707 -1.5707" />
+        <geometry>
+            <cylinder radius="0.1" length="0.05" />
+        </geometry>
+    </collision>
+    <visual name="visual_left">
+        <origin xyz="0 0 0" rpy="0 -1.5707 -1.5707" />
+        <geometry>
+            <cylinder radius="0.1" length="0.05" />
+        </geometry>
+    </visual>
+    <inertial>
+      <mass value="5.0"/>
+      <origin xyz="0.0 0 0" rpy=" 0 0 0"/>
+      <inertia
+          ixx="0.1" ixy="0" ixz="0"
+          iyy="0.1" iyz="0"
+          izz="0.1"
+      />
+    </inertial>
+</link>
 </robot>

Commit message: rotated the robot wheel the opposite side for changing to the right rotating direction

File: urdf/udacity_bot.xacro (robot description, xacro)
@@ -96,5 +96,5 @@
 <link name="right_wheel">
     <collision name="collision_right">
-        <origin xyz="0 0 0" rpy="0 -1.5707 -1.5707" />
+        <origin xyz="0 0 0" rpy="0 1.5707 1.5707" />
         <geometry>
             <cylinder radius="0.1" length="0.05" />
@@ -102,5 +102,5 @@
     </collision>
     <visual name="visual_left">
-        <origin xyz="0 0 0" rpy="0 -1.5707 -1.5707" />
+        <origin xyz="0 0 0" rpy="0 1.5707 1.5707" />
         <geometry>
             <cylinder radius="0.1" length="0.05" />

Commit message: robot urdf created

File: urdf/udacity_bot.xacro (robot description, xacro)
@@ -1,4 +1,5 @@
-<?xml version='1.0'?>
+xml version='1.0'?>
 <robot name="udacity_bot" xmlns:xacro="http://www.ros.org/wiki/xacro">
+  <xacro:include filename="$(find udacity_bot)/urdf/udacity_bot.gazebo" />
   <link name="robot_footprint"></link>
   <joint name="robot_footprint_joint" type="fixed">
@@ -117,3 +118,59 @@
     </inertial>
 </link>
+<link name="camera">
+    <collision name="camera_collision">
+        <origin xyz="0 0 0" rpy="0 0 0" />
+        <geometry>
+            <box size="0.05 0.05 0.05" />
+        </geometry>
+    </collision>
+    <visual name="camera_visual">
+        <origin xyz="0 0 0" rpy="0 0 0" />
+        <geometry>
+            <box size="0.05 0.05 0.05" />
+        </geometry>
+    </visual>
+    <inertial>
+      <mass value="0.2"/>
+      <origin xyz="0.0 0 0" rpy=" 0 0 0"/>
+      <inertia
+          ixx="1e-6" ixy="0" ixz="0"
+          iyy="1e-6" iyz="0"
+          izz="1e-6"
+      />
+    </inertial>
+</link>
+<joint type="fixed" name="camera_joint">
+    <origin xyz="0 0 0.2" rpy="0 0 0"/>
+    <child link="camera"/>
+    <parent link="chassis"/>
+</joint>
+<link name="hokuyo">
+    <collision name="hokuyo_collision">
+        <origin xyz="0 0 0" rpy="0 0 0" />
+        <geometry>
+            <box size="0.1 0.1 0.1" />
+        </geometry>
+    </collision>
+    <visual name="hokuyo_visual">
+        <origin xyz="0 0 0" rpy="0 0 0" />
+        <geometry>
+            <mesh filename="package://udacity_bot/meshes/hokuyo.dae"/>
+        </geometry>
+    </visual>
+    <inertial>
+      <mass value="0.1"/>
+      <origin xyz="0.0 0 0" rpy=" 0 0 0"/>
+      <inertia
+          ixx="1e-6" ixy="0" ixz="0"
+          iyy="1e-6" iyz="0"
+          izz="1e-6"
+      />
+    </inertial>
+</link>
+<joint type="fixed" name="hokuyo_joint">
+    <origin xyz="0.15 0 0.1" rpy="0 0 0"/>
+    <child link="hokuyo"/>
+    <parent link="chassis"/>
+</joint>
 </robot>

Commit message: wrong camera position fixed

File: urdf/udacity_bot.xacro (robot description, xacro)
@@ -142,5 +142,5 @@
 </link>
 <joint type="fixed" name="camera_joint">
-    <origin xyz="0 0 0.2" rpy="0 0 0"/>
+    <origin xyz="0.2 0 0" rpy="0 0 0"/>
     <child link="camera"/>
     <parent link="chassis"/>

Commit message: differential controller plugin fixed

File: urdf/udacity_bot.xacro (robot description, xacro)
@@ -87,5 +87,5 @@
     </inertial>
 </link>
-<joint type="continuous" name="right_heel_hinge">
+<joint type="continuous" name="right_wheel_hinge">
     <origin xyz="0 -0.15 0" rpy="0 0 0"/>
     <child link="right_wheel"/>
